File: steller/steller.kicad_pcb (KiCad board)
At the start: 2 copper layers, 135 x 97.8 mm, 37 parts

Commit message: trrs, reset button.
Parts:
- added B1: , E73:SW_TACT_ALPS_SKQGABE010, F.Cu at (202.6, 97.5)
- added TRRS1: , ceoloide:trrs_pj320a (reversible), F.Cu at (204.4, 87.7)
Changed lines of the file:
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@@
         (pad 24 thru_hole circle (at 13.97 7.62 0) (size 1.7526 1.7526) (drill 1.0922) (layers *.Cu *.SilkS *.Mask) (net 40 "P9"))
       )
+  (footprint "ceoloide:trrs_pj320a (reversible)"
+    (layer "F.Cu")
+    (at 204.37635945 87.69348935 -90)
+    (property "Reference" "TRRS1"
+      (at 0 14.2 -90)
+      (layer "F.SilkS")
+      hide
+      (effects (font (size 1 1) (thickness 0.15)))
+    )
+    (fp_line (start 3.9499999999999997 -2) (end -1.65 -2) (layer "Dwgs.User") (stroke (width 0.15) (type solid)))
+    (fp_line (start -1.65 0) (end -1.65 -2) (layer "Dwgs.User") (stroke (width 0.15) (type solid)))
+    (fp_line (start 3.9499999999999997 0) (end 3.9499999999999997 -2) (layer "Dwgs.User") (stroke (width 0.15) (type solid)))
+    (fp_line (start -1.9 0) (end -1.9 12.1) (layer "Dwgs.User") (stroke (width 0.15) (type solid)))
+    (fp_line (start 4.199999999999999 0) (end 4.199999999999999 12.1) (layer "Dwgs.User") (stroke (width 0.15) (type solid)))
+    (fp_line (start 4.199999999999999 12.1) (end -1.9 12.1) (layer "Dwgs.User") (stroke (width 0.15) (type solid)))
+    (fp_line (start 4.199999999999999 0) (end -1.9 0) (layer "Dwgs.User") (stroke (width 0.15) (type solid)))
+    (pad "" np_thru_hole circle (at -1.15 8.6 -90) (size 1.5 1.5) (drill 1.5) (layers "*.Cu" "*.Mask"))
+    (pad "" np_thru_hole circle (at -1.15 1.6 -90) (size 1.5 1.5) (drill 1.5) (layers "*.Cu" "*.Mask"))
+    (pad "" np_thru_hole circle (at 1.15 8.6 -90) (size 1.5 1.5) (drill 1.5) (layers "*.Cu" "*.Mask"))
+    (pad "" np_thru_hole circle (at 1.15 1.6 -90) (size 1.5 1.5) (drill 1.5) (layers "*.Cu" "*.Mask"))
+    (pad 2 thru_hole oval (at 3.45 3.2 -90) (size 1.6 2.2) (drill oval 0.9 1.5) (layers "*.Cu" "*.Mask") (net 20 "GND"))
+    (pad 3 thru_hole oval (at 3.45 6.2 -90) (size 1.6 2.2) (drill oval 0.9 1.5) (layers "*.Cu" "*.Mask") (net 31 "P1"))
+    (pad 4 thru_hole oval (at 3.45 10.2 -90) (size 1.6 2.2) (drill oval 0.9 1.5) (layers "*.Cu" "*.Mask") (net 20 "GND"))
+    (pad 5 thru_hole oval (at -1.15 11.3 -90) (size 1.6 2.2) (drill oval 0.9 1.5) (layers "*.Cu" "*.Mask") (net 22 "VCC"))
+    (pad 2 thru_hole oval (at -3.45 3.2 -90) (size 1.6 2.2) (drill oval 0.9 1.5) (layers "*.Cu" "*.Mask") (net 20 "GND"))
+    (pad 3 thru_hole oval (at -3.45 6.2 -90) (size 1.6 2.2) (drill oval 0.9 1.5) (layers "*.Cu" "*.Mask") (net 31 "P1"))
+    (pad 4 thru_hole oval (at -3.45 10.2 -90) (size 1.6 2.2) (drill oval 0.9 1.5) (layers "*.Cu" "*.Mask") (net 20 "GND"))
+    (pad 5 thru_hole oval (at 1.15 11.3 -90) (size 1.6 2.2) (drill oval 0.9 1.5) (layers "*.Cu" "*.Mask") (net 22 "VCC"))
+  )
+    (module E73:SW_TACT_ALPS_SKQGABE010 (layer F.Cu)
+        (descr "Low-profile SMD Tactile Switch, https://www.e-switch.com/product-catalog/tact/product-lines/tl3342-series-low-profile-smt-tact-switch")
+        (tags "SPST Tactile Switch")
+        (at 202.63987775 97.54156685 -90)
+        (fp_text reference "B1" (at 0 0) (layer F.SilkS) hide (effects (font (size 1.27 1.27) (thickness 0.15))))
+        (fp_text value "" (at 0 0) (layer F.SilkS) hide (effects (font (size 1.27 1.27) (thickness 0.15))))
+        (fp_line (start 2.75 1.25) (end 1.25 2.75) (layer F.SilkS) (width 0.15))
+        (fp_line (start 2.75 -1.25) (end 1.25 -2.75) (layer F.SilkS) (width 0.15))
+        (fp_line (start 2.75 -1.25) (end 2.75 1.25) (layer F.SilkS) (width 0.15))
+        (fp_line (start -1.25 2.75) (end 1.25 2.75) (layer F.SilkS) (width 0.15))
+        (fp_line (start -1.25 -2.75) (end 1.25 -2.75) (layer F.SilkS) (width 0.15))
+        (fp_line (start -2.75 1.25) (end -1.25 2.75) (layer F.SilkS) (width 0.15))
+        (fp_line (start -2.75 -1.25) (end -1.25 -2.75) (layer F.SilkS) (width 0.15))
+        (fp_line (start -2.75 -1.25) (end -2.75 1.25) (layer F.SilkS) (width 0.15))
+        (pad 1 smd rect (at -3.1 -1.85 -90) (size 1.8 1.1) (layers F.Cu F.Paste F.Mask) (net 20 "GND"))
+        (pad 1 smd rect (at 3.1 -1.85 -90) (size 1.8 1.1) (layers F.Cu F.Paste F.Mask) (net 20 "GND"))
+        (pad 2 smd rect (at -3.1 1.85 -90) (size 1.8 1.1) (layers F.Cu F.Paste F.Mask) (net 21 "RST"))
+        (pad 2 smd rect (at 3.1 1.85 -90) (size 1.8 1.1) (layers F.Cu F.Paste F.Mask) (net 21 "RST"))
+    )
   (gr_line (start 90 107.43814297317073) (end 90 53.610249293684205) (angle 90) (layer Edge.Cuts) (width 0.15))
 (gr_line (start 91.34197774605971 51.11005686313935) (end 108.66626471113908 39.6213191915604) (angle 90) (layer Edge.Cuts) (width 0.15))
